File: src/bin_clock_kicad/bin_clock.sch (KiCad schematic (older format))
At the start: 35 parts, among them J1 Screw_Terminal_1x02, J10 CONN_01X02, J2 CONN_01X02, J3 CONN_01X04, J4 CONN_01X03, J5 CONN_01X03, J6 CONN_02X03, J7 CONN_01X02, J8 CONN_01X02, J9 CONN_01X02, U1 ATMEGA324A-PU, Y1 Crystal

Commit message: added missing sone button
Parts:
- added J?: CONN_01X02, symbol CONN_01X02
- added R? (x2): R, symbol R
Connections:
- net +5V: now also R?.1, R?.1
- net GND: now also J?.2 (P2)
- net at J5.2 (P2), U1.28 ((PCINT22/TOSC1)PC6): now also R?.2
- net at U1.29 ((PCINT23/TOSC2)PC7): now also J?.1 (P1), R?.2
- net at D?.1 (VDD): now also D?.1 (VDD), D?.1 (VDD), D?.1 (VDD) (x2)
- net at D?.2 (DOUT): now also D?.4 (DIN) (x7)
- net at D?.3 (VSS): now also D?.3 (VSS), D?.3 (VSS), D?.3 (VSS) (x2)
Other:
- note added: "SHUT UP\nALARM\n"
- moved on the sheet: D?

Commit message: added all leds
Parts:
- added D13, D14, D15, D16, D17, D18, D19, D20, D21, D22, D23, D24, D25, D26, D27: 1655, FCI_1655, symbol 1655
- gave numbers to parts that had none: 17
- renumbered J8 to J10, J9 to J11, J10 to J12, J3 to J5, J4 to J6, J5 to J7, J6 to J8, J7 to J9, R2 to R4, R3 to R5, R4 to R6, R5 to R7
Connections:
- net +5V: now also D10.1 (VDD), D11.1 (VDD), D12.1 (VDD), D4.1 (VDD), D5.1 (VDD), D6.1 (VDD), D7.1 (VDD), D8.1 (VDD), D9.1 (VDD), D13.1 (VDD), D14.1 (VDD), D15.1 (VDD), D16.1 (VDD), D17.1 (VDD), D18.1 (VDD), D19.1 (VDD), D20.1 (VDD), D21.1 (VDD), D22.1 (VDD), D23.1 (VDD), D24.1 (VDD), D25.1 (VDD), D26.1 (VDD), D27.1 (VDD)
- net GND: now also D10.3 (VSS), D11.3 (VSS), D12.3 (VSS), D4.3 (VSS), D5.3 (VSS), D6.3 (VSS), D7.3 (VSS), D8.3 (VSS), D9.3 (VSS), D13.3 (VSS), D14.3 (VSS), D15.3 (VSS), D16.3 (VSS), D17.3 (VSS), D18.3 (VSS), D19.3 (VSS), D20.3 (VSS), D21.3 (VSS), D22.3 (VSS), D23.3 (VSS), D24.3 (VSS), D25.3 (VSS), D26.3 (VSS), D27.3 (VSS)
- net at J7.2 (P2), R2.2, U1.28 ((PCINT22/TOSC1)PC6): now also D4.4 (DIN)
- net at D12.2 (DOUT): now also D13.4 (DIN)
- net at D12.4 (DIN): now also D11.2 (DOUT)
- new net: D13.2 (DOUT), D14.4 (DIN)
- new net: D14.2 (DOUT), D15.4 (DIN)
- new net: D15.2 (DOUT), D16.4 (DIN)
- new net: D19.2 (DOUT), D20.4 (DIN)
- new net: D20.2 (DOUT), D21.4 (DIN)
- new net: D21.2 (DOUT), D22.4 (DIN)
- new net: D22.2 (DOUT), D23.4 (DIN)
- new net: D23.2 (DOUT), D24.4 (DIN)
- new net: D24.2 (DOUT), D25.4 (DIN)
- new net: D25.2 (DOUT), D26.4 (DIN)
- new net: D26.2 (DOUT), D27.4 (DIN)
Other:
- note added: "RESET BTN"
