File: src/bin_clock_kicad/bin_clock.sch (KiCad schematic (older format))
At the start: 52 parts, among them J1 Screw_Terminal_1x02, J10 CONN_01X02, J11 CONN_01X02, J12 CONN_01X02, J13 CONN_01X02, J2 CONN_01X02, J3 TEST_1P, J4 TEST_1P, J5 CONN_01X04, J6 CONN_01X03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

Commit message: pcb rework needed
Parts:
- removed J3, J4: TEST_1P, symbol TEST_1P
- added U?: ATMEGA328P-AU, TQFP32, symbol ATMEGA328P-AU
- 5k1: renamed from R3; footprint (none) -> Resistors_SMD:R_0603_HandSoldering
- C1, C2, C3, C4, C5, C6: footprint (none) -> Capacitors_SMD:C_0603_HandSoldering
- J1: footprint (none) -> Connectors_Terminal_Blocks:TerminalBlock_Pheonix_MPT-2.54mm_2pol
- J10, J11, J12, J13, J9: footprint (none) -> Pin_Headers:Pin_Header_Angled_1x02_Pitch2.54mm
- J2: footprint (none) -> Pin_Headers:Pin_Header_Angled_1x01_Pitch2.54mm
- J5: footprint (none) -> Pin_Headers:Pin_Header_Angled_1x04_Pitch2.54mm
- J6, J7: footprint (none) -> Pin_Headers:Pin_Header_Angled_1x03_Pitch2.54mm
- J8: footprint (none) -> Pin_Headers:Pin_Header_Angled_2x03_Pitch2.54mm
- R1, R2, R4, R5, R6, R7: footprint (none) -> Resistors_SMD:R_0603_HandSoldering
- Y1: footprint (none) -> Crystals:Crystal_HC49-U_Horizontal
Changed lines of the file:
@@
 LIBS:valves
 LIBS:1655
+LIBS:ATMEGA328P-AU
 LIBS:bin_clock-cache
 EELAYER 25 0
@@
 F 0 "R4" V 6030 1500 50  0000 C CNN
 F 1 "R" V 5950 1500 50  0000 C CNN
-F 2 "" V 5880 1500 50  0001 C CNN
+F 2 "Resistors_SMD:R_0603_HandSoldering" V 5880 1500 50  0001 C CNN
 F 3 "" H 5950 1500 50  0001 C CNN
 	1    5950 1500
@@
 F 0 "R5" V 6330 1500 50  0000 C CNN
 F 1 "R" V 6250 1500 50  0000 C CNN
-F 2 "" V 6180 1500 50  0001 C CNN
+F 2 "Resistors_SMD:R_0603_HandSoldering" V 6180 1500 50  0001 C CNN
 F 3 "" H 6250 1500 50  0001 C CNN
 	1    6250 1500
@@
 F 0 "R6" V 6580 1500 50  0000 C CNN
 F 1 "R" V 6500 1500 50  0000 C CNN
-F 2 "" V 6430 1500 50  0001 C CNN
+F 2 "Resistors_SMD:R_0603_HandSoldering" V 6430 1500 50  0001 C CNN
 F 3 "" H 6500 1500 50  0001 C CNN
 	1    6500 1500
@@
 F 0 "R7" V 6830 1500 50  0000 C CNN
 F 1 "R" V 6750 1500 50  0000 C CNN
-F 2 "" V 6680 1500 50  0001 C CNN
+F 2 "Resistors_SMD:R_0603_HandSoldering" V 6680 1500 50  0001 C CNN
 F 3 "" H 6750 1500 50  0001 C CNN
 	1    6750 1500
@@
 F 0 "R1" V 2030 1800 50  0000 C CNN
 F 1 "R" V 1950 1800 50  0000 C CNN
-F 2 "" V 1880 1800 50  0001 C CNN
+F 2 "Resistors_SMD:R_0603_HandSoldering" V 1880 1800 50  0001 C CNN
 F 3 "" H 1950 1800 50  0001 C CNN
 	1    1950 1800
@@
 $EndComp
 $Comp
-L GND #PWR1
+L GND #PWR01
 U 1 1 5931C3B0
 P 3150 5900
-F 0 "#PWR1" H 3150 5650 50  0001 C CNN
+F 0 "#PWR01" H 3150 5650 50  0001 C CNN
 F 1 "GND" H 3150 5750 50  0000 C CNN
 F 2 "" H 3150 5900 50  0001 C CNN
@@
 $EndComp
 $Comp
-L +5V #PWR2
+L +5V #PWR02
 U 1 1 5931C472
 P 3250 1100
-F 0 "#PWR2" H 3250 950 50  0001 C CNN
+F 0 "#PWR02" H 3250 950 50  0001 C CNN
 F 1 "+5V" H 3250 1240 50  0000 C CNN
 F 2 "" H 3250 1100 50  0001 C CNN
@@
 F 0 "J1" H 1200 3850 50  0000 C TNN
 F 1 "Screw_Terminal_1x02" V 1050 3600 50  0000 C TNN
-F 2 "" H 1200 3375 50  0001 C CNN
+F 2 "Connectors_Terminal_Blocks:TerminalBlock_Pheonix_MPT-2.54mm_2pol" H 1200 3375 50  0001 C CNN
 F 3 "" H 1175 3600 50  0001 C CNN
 	1    1200 3600
@@
 F 0 "J6" H 5400 4950 50  0000 C CNN
 F 1 "CONN_01X03" V 5500 4750 50  0000 C CNN
-F 2 "" H 5400 4750 50  0001 C CNN
+F 2 "Pin_Headers:Pin_Header_Angled_1x03_Pitch2.54mm" H 5400 4750 50  0001 C CNN
 F 3 "" H 5400 4750 50  0001 C CNN
 	1    5400 4750
@@
 F 0 "Y1" H 2150 2700 50  0000 C CNN
 F 1 "Crystal" H 2150 2400 50  0000 C CNN
-F 2 "" H 2150 2550 50  0001 C CNN
+F 2 "Crystals:Crystal_HC49-U_Horizontal" H 2150 2550 50  0001 C CNN
 F 3 "" H 2150 2550 50  0001 C CNN
 	1    2150 2550
@@
 F 0 "C3" H 1775 2450 50  0000 L CNN
 F 1 "C" H 1775 2250 50  0000 L CNN
-F 2 "" H 1788 2200 50  0001 C CNN
+F 2 "Capacitors_SMD:C_0603_HandSoldering" H 1788 2200 50  0001 C CNN
 F 3 "" H 1750 2350 50  0001 C CNN
 	1    1750 2350
@@
 F 0 "C4" H 1775 2850 50  0000 L CNN
 F 1 "C" H 1775 2650 50  0000 L CNN
-F 2 "" H 1788 2600 50  0001 C CNN
+F 2 "Capacitors_SMD:C_0603_HandSoldering" H 1788 2600 50  0001 C CNN
 F 3 "" H 1750 2750 50  0001 C CNN
 	1    1750 2750
@@
 F 0 "J2" H 2600 1650 50  0000 C CNN
 F 1 "CONN_01X02" V 2700 1500 50  0000 C CNN
-F 2 "" H 2600 1500 50  0001 C CNN
+F 2 "Pin_Headers:Pin_Header_Angled_1x01_Pitch2.54mm" H 2600 1500 50  0001 C CNN
 F 3 "" H 2600 1500 50  0001 C CNN
 	1    2600 1500
@@
 F 0 "J9" H 7400 1900 50  0000 C CNN
 F 1 "CONN_01X02" V 7500 1750 50  0000 C CNN
-F 2 "" H 7400 1750 50  0001 C CNN
+F 2 "Pin_Headers:Pin_Header_Angled_1x02_Pitch2.54mm" H 7400 1750 50  0001 C CNN
 F 3 "" H 7400 1750 50  0001 C CNN
 	1    7400 1750
@@
 F 0 "J10" H 7400 2200 50  0000 C CNN
 F 1 "CONN_01X02" V 7500 2050 50  0000 C CNN
-F 2 "" H 7400 2050 50  0001 C CNN
+F 2 "Pin_Headers:Pin_Header_Angled_1x02_Pitch2.54mm" H 7400 2050 50  0001 C CNN
 F 3 "" H 7400 2050 50  0001 C CNN
 	1    7400 2050
@@
 F 0 "J11" H 7400 2500 50  0000 C CNN
 F 1 "CONN_01X02" V 7500 2350 50  0000 C CNN
-F 2 "" H 7400 2350 50  0001 C CNN
+F 2 "Pin_Headers:Pin_Header_Angled_1x02_Pitch2.54mm" H 7400 2350 50  0001 C CNN
 F 3 "" H 7400 2350 50  0001 C CNN
 	1    7400 2350
@@
 F 0 "J12" H 7400 2800 50  0000 C CNN
 F 1 "CONN_01X02" V 7500 2650 50  0000 C CNN
-F 2 "" H 7400 2650 50  0001 C CNN
+F 2 "Pin_Headers:Pin_Header_Angled_1x02_Pitch2.54mm" H 7400 2650 50  0001 C CNN
 F 3 "" H 7400 2650 50  0001 C CNN
 	1    7400 2650
@@
 F 0 "J5" H 5400 3850 50  0000 C CNN
 F 1 "CONN_01X04" V 5500 3600 50  0000 C CNN
-F 2 "" H 5400 3600 50  0001 C CNN
+F 2 "Pin_Headers:Pin_Header_Angled_1x04_Pitch2.54mm" H 5400 3600 50  0001 C CNN
 F 3 "" H 5400 3600 50  0001 C CNN
 	1    5400 3600
@@
 F 0 "J7" H 5450 3000 50  0000 C CNN
 F 1 "CONN_01X03" V 5550 2800 50  0000 C CNN
-F 2 "" H 5450 2800 50  0001 C CNN
+F 2 "Pin_Headers:Pin_Header_Angled_1x03_Pitch2.54mm" H 5450 2800 50  0001 C CNN
 F 3 "" H 5450 2800 50  0001 C CNN
 	1    5450 2800
@@
 F 0 "J8" H 5800 5600 50  0000 C CNN
 F 1 "CONN_02X03" H 5800 5200 50  0000 C CNN
-F 2 "" H 5800 4200 50  0001 C CNN
+F 2 "Pin_Headers:Pin_Header_Angled_2x03_Pitch2.54mm" H 5800 4200 50  0001 C CNN
 F 3 "" H 5800 4200 50  0001 C CNN
 	1    5800 5400
@@
 F 0 "C1" H 1175 2550 50  0000 L CNN
 F 1 "C" H 1175 2350 50  0000 L CNN
-F 2 "" H 1188 2300 50  0001 C CNN
+F 2 "Capacitors_SMD:C_0603_HandSoldering" H 1188 2300 50  0001 C CNN
 F 3 "" H 1150 2450 50  0001 C CNN
 	1    1150 2450
@@
 F 0 "C2" H 1175 2800 50  0000 L CNN
 F 1 "C" H 1175 2600 50  0000 L CNN
-F 2 "" H 1188 2550 50  0001 C CNN
+F 2 "Capacitors_SMD:C_0603_HandSoldering" H 1188 2550 50  0001 C CNN
 F 3 "" H 1150 2700 50  0001 C CNN
 	1    1150 2700
-	0    1    1    0
-$EndComp
-$Comp
-L TEST_1P J4
-U 1 1 5931D28C
-P 4550 1950
-F 0 "J4" H 4550 2220 50  0000 C CNN
-F 1 "TEST_1P" H 4550 2150 50  0000 C CNN
-F 2 "" H 4750 1950 50  0001 C CNN
-F 3 "" H 4750 1950 50  0001 C CNN
-	1    4550 1950
-	0    1    1    0
-$EndComp
-$Comp
-L TEST_1P J3
-U 1 1 5931D771
-P 4500 5550
-F 0 "J3" H 4500 5820 50  0000 C CNN
-F 1 "TEST_1P" H 4500 5750 50  0000 C CNN
-F 2 "" H 4700 5550 50  0001 C CNN
-F 3 "" H 4700 5550 50  0001 C CNN
-	1    4500 5550
 	0    1    1    0
 $EndComp
@@
 F 0 "R2" V 4930 2550 50  0000 C CNN
 F 1 "R" V 4850 2550 50  0000 C CNN
-F 2 "" V 4780 2550 50  0001 C CNN
+F 2 "Resistors_SMD:R_0603_HandSoldering" V 4780 2550 50  0001 C CNN
 F 3 "" H 4850 2550 50  0001 C CNN
 	1    4850 2550
@@
 F 0 "J13" H 7400 3450 50  0000 C CNN
 F 1 "CONN_01X02" V 7500 3300 50  0000 C CNN
-F 2 "" H 7400 3300 50  0001 C CNN
+F 2 "Pin_Headers:Pin_Header_Angled_1x02_Pitch2.54mm" H 7400 3300 50  0001 C CNN
 F 3 "" H 7400 3300 50  0001 C CNN
 	1    7400 3300
@@
 $EndComp
 $Comp
-L R R3
+L R 5k1
 U 1 1 5932D3F9
 P 5700 1500
-F 0 "R3" V 5780 1500 50  0000 C CNN
+F 0 "5k1" V 5780 1500 50  0000 C CNN
 F 1 "R" V 5700 1500 50  0000 C CNN
-F 2 "" V 5630 1500 50  0001 C CNN
+F 2 "Resistors_SMD:R_0603_HandSoldering" V 5630 1500 50  0001 C CNN
 F 3 "" H 5700 1500 50  0001 C CNN
 	1    5700 1500
@@
 Connection ~ 3250 1100
 Wire Wire Line
-	4350 1950 4550 1950
-Wire Wire Line
-	4350 5050 4500 5050
-Wire Wire Line
-	4500 5050 4500 5550
-Wire Wire Line
 	4850 2400 5050 2400
 Connection ~ 5050 2400
@@
 Connection ~ 5700 3250
 Wire Wire Line
-	13450 3950 13600 3950
+	13600 3950 13450 3950
 Wire Wire Line
 	13600 2600 13600 7000
@@
 Connection ~ 17050 7000
 Wire Wire Line
-	20200 6100 20250 6100
+	20250 6100 20200 6100
 Wire Wire Line
 	20250 3400 20250 6900
@@
 F 0 "C5" H 13575 2550 50  0000 L CNN
 F 1 "C" H 13575 2350 50  0000 L CNN
-F 2 "" H 13588 2300 50  0001 C CNN
+F 2 "Capacitors_SMD:C_0603_HandSoldering" H 13588 2300 50  0001 C CNN
 F 3 "" H 13550 2450 50  0001 C CNN
 	1    13550 2450
@@
 F 0 "C6" H 13825 2550 50  0000 L CNN
 F 1 "C" H 13825 2350 50  0000 L CNN
-F 2 "" H 13838 2300 50  0001 C CNN
+F 2 "Capacitors_SMD:C_0603_HandSoldering" H 13838 2300 50  0001 C CNN
 F 3 "" H 13800 2450 50  0001 C CNN
 	1    13800 2450
@@
 Connection ~ 13650 3000
 Connection ~ 13700 2300
+$Comp
+L ATMEGA328P-AU U?
+U 1 1 59332C92
+P 3350 7950
+F 0 "U?" H 2600 9200 50  0000 L BNN
+F 1 "ATMEGA328P-AU" H 3750 6550 50  0000 L BNN
+F 2 "TQFP32" H 3350 7950 50  0001 C CIN
+F 3 "" H 3350 7950 50  0001 C CNN
+	1    3350 7950
+	1    0    0    -1
+$EndComp
 $EndSCHEMATC
