File: src/bin_clock_eagle/main_clock_board.brd (EAGLE design)
At the start: 160 x 100 mm, 51 parts, among them U1 ATMEGA328P-AU, U2 DS1307Z+

Commit message: added vcc gnd pins
Connections:
- net N$48 renamed GND
- net N$49 renamed VCC
Changed lines of the file:
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@@
 <wire x1="80.01" y1="19.05" x2="79.883" y2="19.05" width="0.1524" layer="1"/>
 </signal>
-<signal name="N$48">
+<signal name="GND">
 <contactref element="C1" pad="2"/>
 <contactref element="C2" pad="2"/>
@@
 <wire x1="79.81465" y1="25.436846875" x2="79.465809375" y2="25.7856875" width="0.1524" layer="1"/>
 </signal>
-<signal name="N$49">
+<signal name="VCC">
 <contactref element="C3" pad="2"/>
 <contactref element="C4" pad="1"/>
