File: src/bin_clock_eagle/main_clock_board.sch (EAGLE design)
At the start: 51 parts, among them U1 ATMEGA328P-AU, U2 DS1307Z+

Commit message: added part values
Parts:
- C1, C2: value (none) -> 22p
- C3, C4: value (none) -> 100n
- Q1: value (none) -> 32.768 khz
- Q2: value (none) -> 16Mhz
- R1, R26, R27: value (none) -> 10k
- R13, R18, R23, R28, R3, R5: value (none) -> 5k
Other:
- moved on the sheet: D10, D11, D12, D13, D14, D15, D16, D17, D18, D19, D20, D21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

Commit message: pcb size rework
Parts:
- C1, C2: value 22p -> (none)
- C3, C4: value 100n -> (none)
- Q1: value 32.768 khz -> (none)
- Q2: value 16Mhz -> (none)
- R1, R26, R27: value 10k -> (none)
- R13, R18, R23, R28, R3, R5: value 5k -> (none)
Other:
- moved on the sheet: D10, D11, D12, D13, D14, D15, D16, D17, D18, D19, D20, D21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
