File: src/bin_clock_eagle/main_clock_board.sch (EAGLE design)
At the start: 51 parts, among them U1 ATMEGA328P-AU, U2 DS1307Z+

Commit message: added gound planes
Parts:
- removed Q1: (no value), adafruit:CRYSTALHC49S
- removed R25: (no value), adafruit:R-US_R0603
- removed U2: DS1307Z+, DS1307Z_:DS1307Z+
- added C10, C11, C12, C13, C14, C15, C16, C17, C18, C19, C20, C21, C22, C23, C24, C25, C26, C27, C28, C29, C30, C5, C6, C7, C8, C9: 100n, adafruit:C-US025-024X044
- added J9: (no value), Wurth_Elektronik_Electromechanic_Board_to_Board_Connectors_rev16c:61300211121
- added R4, R7: 5k, adafruit:R-US_R0603
- added R6: 220, adafruit:R-US_R0603
- added U$1: DS3231, DS3231:DS3231
- C1, C2: value (none) -> 22p
- C3, C4: value (none) -> 100n
- Q2: value (none) -> 16mhz
- R1, R26, R27: value (none) -> 10k
- R13, R18, R2, R23, R28, R3, R5: value (none) -> 5k
Connections:
- removed net N$22: R25.1, U2.VBAT
- new net N$15: R2.1, U$1.RST
- net GND: now also C10.2, C11.2, C12.2, C13.2, C14.2, C15.2, C16.2, C17.2, C18.2, C19.2, C20.2, C21.2, C22.2, C23.2, C24.2, C25.2, C26.2, C27.2, C28.2, C29.2, C30.2, C5.2, C6.2, C7.2, C8.2, C9.2, J9.1, U$1.GND, U$1.P$1, U$1.P$2, U$1.P$3, U$1.P$4, U$1.P$5, U$1.P$6, U$1.P$7, U$1.P$8; no longer U2.GND
- net N$10: now also U$1.SCL; no longer U2.SCL
- net N$2: now also U$1.SDA; no longer U2.SDA
- net N$43: now also R4.1, U$1.32KHZ; no longer Q1.2, U2.X1
- net N$44: now also J9.2, R6.1, U$1.VBAT; no longer Q1.1, U2.X2
- net N$45: now also R7.1, U$1.INT; no longer R2.1, U2.SQW/OUT
- net VCC: now also C10.1, C11.1, C12.1, C13.1, C14.1, C15.1, C16.1, C17.1, C18.1, C19.1, C20.1, C21.1, C22.1, C23.1, C24.1, C25.1, C26.1, C27.1, C28.1, C29.1, C30.1, C5.1, C6.1, C7.1, C8.1, C9.1, R4.2, R6.2, R7.2, U$1.VCC; no longer R25.2, U2.VCC
Other:
- note added: "RTC BATT"
- moved on the sheet: D10, D11, D12, D13, D14, D15, D16, D17, D18, D19, D20, D21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
